Commit message: Add files via upload

File: simulation/robot_arm_description/urdf/robot_arm.urdf.xacro (robot description, xacro)
@@ -0,0 +1,284 @@
+<?xml version="1.0"?>
+<robot name="color_sorting_arm"
+       xmlns:xacro="http://www.ros.org/wiki/xacro">
+  <!-- ========================================= -->
+  <!-- ROBOT DIMENSIONS (metres)                 -->
+  <!-- ========================================= -->
+  <xacro:property name="base_height" value="0.10"/>
+  <xacro:property name="upper_arm_length" value="0.105"/>
+  <xacro:property name="forearm_length" value="0.127"/>
+  <xacro:property name="wrist_length" value="0.070"/>
+  <!-- ========================================= -->
+  <!-- BASE LINK                                 -->
+  <!-- ========================================= -->
+  <link name="base_link">
+    <visual>
+      <origin xyz="0 0 0.015" rpy="0 0 0"/>
+      <geometry>
+        <box size="0.15 0.15 0.03"/>
+      </geometry>
+      <material name="black">
+        <color rgba="0.12 0.12 0.12 1"/>
+      </material>
+    </visual>
+    <collision>
+  <origin xyz="0 0 0.015" rpy="0 0 0"/>
+  <geometry>
+    <box size="0.15 0.15 0.03"/>
+  </geometry>
+</collision>
+  </link>
+  <!-- ========================================= -->
+  <!-- J1: BASE ROTATION                         -->
+  <!-- ========================================= -->
+  <link name="base_rotation_link">
+    <visual>
+      <origin xyz="0 0 0.05" rpy="0 0 0"/>
+      <geometry>
+        <cylinder radius="0.04" length="0.10"/>
+      </geometry>
+      <material name="gray">
+        <color rgba="0.5 0.5 0.5 1"/>
+      </material>
+    </visual>
+    <collision>
+  <origin xyz="0 0 0.05" rpy="0 0 0"/>
+  <geometry>
+    <cylinder radius="0.04" length="0.10"/>
+  </geometry>
+</collision>
+  </link>
+  <joint name="joint1" type="revolute">
+    <parent link="base_link"/>
+    <child link="base_rotation_link"/>
+    <origin xyz="0 0 0.03" rpy="0 0 0"/>
+    <axis xyz="0 0 1"/>
+    <limit lower="-1.57"
+           upper="1.57"
+           effort="10"
+           velocity="1"/>
+  </joint>
+  <!-- ========================================= -->
+  <!-- J2: SHOULDER                              -->
+  <!-- ========================================= -->
+  <link name="upper_arm_link">
+    <visual>
+      <origin xyz="0 0 ${upper_arm_length / 2}"
+              rpy="0 0 0"/>
+      <geometry>
+        <box size="0.035 0.035 ${upper_arm_length}"/>
+      </geometry>
+      <material name="blue">
+        <color rgba="0.1 0.3 0.9 1"/>
+      </material>
+    </visual>
+      <!-- ADD THIS COLLISION BLOCK -->
+  <collision>
+    <origin xyz="0 0 ${upper_arm_length / 2}"
+            rpy="0 0 0"/>
+    <geometry>
+      <box size="0.035 0.035 ${upper_arm_length}"/>
+    </geometry>
+  </collision>
+  </link>
+  <joint name="joint2" type="revolute">
+    <parent link="base_rotation_link"/>
+    <child link="upper_arm_link"/>
+    <origin xyz="0 0 ${base_height - 0.03}"
+            rpy="0 0 0"/>
+    <axis xyz="0 1 0"/>
+    <limit lower="-1.57"
+           upper="1.57"
+           effort="10"
+           velocity="1"/>
+  </joint>
+  <!-- ========================================= -->
+  <!-- J3: ELBOW                                 -->
+  <!-- ========================================= -->
+  <link name="forearm_link">
+    <visual>
+      <origin xyz="0 0 ${forearm_length / 2}"
+              rpy="0 0 0"/>
+      <geometry>
+        <box size="0.03 0.03 ${forearm_length}"/>
+      </geometry>
+      <material name="green">
+        <color rgba="0.1 0.7 0.3 1"/>
+      </material>
+    </visual>
+    <collision>
+  <origin xyz="0 0 ${forearm_length / 2}" rpy="0 0 0"/>
+  <geometry>
+    <box size="0.03 0.03 ${forearm_length}"/>
+  </geometry>
+</collision>
+  </link>
+  <joint name="joint3" type="revolute">
+    <parent link="upper_arm_link"/>
+    <child link="forearm_link"/>
+    <origin xyz="0 0 ${upper_arm_length}"
+            rpy="0 0 0"/>
+    <axis xyz="0 1 0"/>
+    <limit lower="-1.57"
+           upper="1.57"
+           effort="10"
+           velocity="1"/>
+  </joint>
+  <!-- ========================================= -->
+  <!-- J4: WRIST BENDING                         -->
+  <!-- ========================================= -->
+  <link name="wrist_link">
+    <visual>
+      <origin xyz="0 0 ${wrist_length / 2}"
+              rpy="0 0 0"/>
+      <geometry>
+        <box size="0.025 0.025 ${wrist_length}"/>
+      </geometry>
+      <material name="orange">
+        <color rgba="1.0 0.5 0.1 1"/>
+      </material>
+    </visual>
+    <collision>
+  <origin xyz="0 0 ${wrist_length / 2}" rpy="0 0 0"/>
+  <geometry>
+    <box size="0.025 0.025 ${wrist_length}"/>
+  </geometry>
+</collision>
+  </link>
+  <joint name="joint4" type="revolute">
+    <parent link="forearm_link"/>
+    <child link="wrist_link"/>
+    <origin xyz="0 0 ${forearm_length}"
+            rpy="0 0 0"/>
+    <axis xyz="0 1 0"/>
+    <limit lower="-1.57"
+           upper="1.57"
+           effort="10"
+           velocity="1"/>
+  </joint>
+  <!-- ========================================= -->
+  <!-- J5: GRIPPER ROTATION                      -->
+  <!-- ========================================= -->
+  <link name="gripper_mount_link">
+    <visual>
+      <origin xyz="0 0 0.02" rpy="0 0 0"/>
+      <geometry>
+        <cylinder radius="0.025" length="0.04"/>
+      </geometry>
+      <material name="silver">
+        <color rgba="0.7 0.7 0.7 1"/>
+      </material>
+    </visual>
+    <collision>
+  <origin xyz="0 0 0.02" rpy="0 0 0"/>
+  <geometry>
+    <cylinder radius="0.025" length="0.04"/>
+  </geometry>
+</collision>
+  </link>
+  <joint name="joint5" type="revolute">
+    <parent link="wrist_link"/>
+    <child link="gripper_mount_link"/>
+    <origin xyz="0 0 ${wrist_length}"
+            rpy="0 0 0"/>
+    <axis xyz="0 0 1"/>
+    <limit lower="-1.57"
+           upper="1.57"
+           effort="10"
+           velocity="1"/>
+  </joint>
+  <!-- ========================================= -->
+  <!-- FIXED GRIPPER FINGER                      -->
+  <!-- ========================================= -->
+  <link name="fixed_finger_link">
+    <visual>
+      <origin xyz="0 -0.025 0.055"
+              rpy="0 0 0"/>
+      <geometry>
+        <box size="0.012 0.012 0.07"/>
+      </geometry>
+      <material name="gray_finger">
+        <color rgba="0.6 0.6 0.6 1"/>
+      </material>
+    </visual>
+    <collision>
+  <origin xyz="0 -0.025 0.055" rpy="0 0 0"/>
+  <geometry>
+    <box size="0.012 0.012 0.07"/>
+  </geometry>
+</collision>
+  </link>
+  <joint name="fixed_finger_joint" type="fixed">
+    <parent link="gripper_mount_link"/>
+    <child link="fixed_finger_link"/>
+    <origin xyz="0 0 0.02" rpy="0 0 0"/>
+  </joint>
+  <!-- ========================================= -->
+  <!-- J6: GRIPPER OPENING AND CLOSING           -->
+  <!-- ========================================= -->
+  <link name="moving_finger_link">
+    <visual>
+      <origin xyz="0 0 0.035"
+              rpy="0 0 0"/>
+      <geometry>
+        <box size="0.012 0.012 0.07"/>
+      </geometry>
+      <material name="gray_moving_finger">
+        <color rgba="0.6 0.6 0.6 1"/>
+      </material>
+    </visual>
+    <collision>
+  <origin xyz="0 0 0.035" rpy="0 0 0"/>
+  <geometry>
+    <box size="0.012 0.012 0.07"/>
+  </geometry>
+</collision>
+  </link>
+  <joint name="joint6" type="prismatic">
+    <parent link="gripper_mount_link"/>
+    <child link="moving_finger_link"/>
+    <origin xyz="0 0.025 0.04"
+            rpy="0 0 0"/>
+    <axis xyz="0 -1 0"/>
+    <limit lower="0.0"
+           upper="0.035"
+           effort="10"
+           velocity="0.05"/>
+  </joint>
+<!-- Simulated hardware for MoveIt testing -->
+<ros2_control name="SimulatedArm" type="system">
+  <hardware>
+    <plugin>mock_components/GenericSystem</plugin>
+  </hardware>
+  <joint name="joint1">
+    <command_interface name="position"/>
+    <state_interface name="position"/>
+    <state_interface name="velocity"/>
+  </joint>
+  <joint name="joint2">
+    <command_interface name="position"/>
+    <state_interface name="position"/>
+    <state_interface name="velocity"/>
+  </joint>
+  <joint name="joint3">
+    <command_interface name="position"/>
+    <state_interface name="position"/>
+    <state_interface name="velocity"/>
+  </joint>
+  <joint name="joint4">
+    <command_interface name="position"/>
+    <state_interface name="position"/>
+    <state_interface name="velocity"/>
+  </joint>
+  <joint name="joint5">
+    <command_interface name="position"/>
+    <state_interface name="position"/>
+    <state_interface name="velocity"/>
+  </joint>
+  <joint name="joint6">
+    <command_interface name="position"/>
+    <state_interface name="position"/>
+    <state_interface name="velocity"/>
+  </joint>
+</ros2_control>
+</robot>
